File: BPS-Amperes.kicad_sch (KiCad schematic)
At the start: 55 parts, among them J1 ShuntConn, J2 LeaderConn, J3 Conn_01x04, U1 INA186A3IDDFT, U2 RO-123.3S_HP, U3 LTC6820, U4 HX1188FNL, U5 REF1930AIDDCT, U6 LTC2315, U7 OPA2196

Commit message: datasheets & annotations
Parts:
- D2, D3: footprint (none) -> Diode_SMD:D_0805_2012Metric
Changed lines of the file:
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@@
   (symbol (lib_id "Connector:TestPoint") (at 62.23 60.96 180) (unit 1)
     (in_bom yes) (on_board yes)
-    (property "Reference" "TP2" (id 0) (at 63.5 63.5 0)
+    (property "Reference" "TP2" (id 0) (at 60.96 66.04 0)
       (effects (font (size 1.27 1.27)) (justify right))
     )
-    (property "Value" "GNDPWR_TP" (id 1) (at 63.5 66.04 0)
+    (property "Value" "GNDPWR_TP" (id 1) (at 60.96 68.58 0)
       (effects (font (size 1.27 1.27)) (justify right))
     )
@@
       (effects (font (size 1.27 1.27)) hide)
     )
-    (property "Footprint" "" (id 2) (at 44.45 50.8 0)
-      (effects (font (size 1.27 1.27)) hide)
-    )
-    (property "Datasheet" "~" (id 3) (at 44.45 50.8 0)
+    (property "Footprint" "Diode_SMD:D_0805_2012Metric" (id 2) (at 44.45 50.8 0)
+      (effects (font (size 1.27 1.27)) hide)
+    )
+    (property "Datasheet" "https://fscdn.rohm.com/en/products/databook/datasheet/discrete/diode/schottky_barrier/rb061qs-20-e.pdf" (id 3) (at 44.45 50.8 0)
       (effects (font (size 1.27 1.27)) hide)
     )
@@
       (effects (font (size 1.27 1.27)) hide)
     )
-    (property "Datasheet" "~" (id 3) (at 97.79 91.44 0)
+    (property "Datasheet" "https://www.mouser.com/ProductDetail/963-BK2125LM182-T" (id 3) (at 97.79 91.44 0)
       (effects (font (size 1.27 1.27)) hide)
     )
@@
       (effects (font (size 1.27 1.27)) hide)
     )
-    (property "Datasheet" "~" (id 3) (at 97.79 87.63 0)
+    (property "Datasheet" "https://www.mouser.com/ProductDetail/963-BK2125LM182-T" (id 3) (at 97.79 87.63 0)
       (effects (font (size 1.27 1.27)) hide)
     )
@@
       (effects (font (size 1.27 1.27)) (justify left))
     )
-    (property "Footprint" "" (id 2) (at 138.43 167.64 0)
-      (effects (font (size 1.27 1.27)) hide)
-    )
-    (property "Datasheet" "~" (id 3) (at 138.43 167.64 0)
+    (property "Footprint" "Diode_SMD:D_0805_2012Metric" (id 2) (at 138.43 167.64 0)
+      (effects (font (size 1.27 1.27)) hide)
+    )
+    (property "Datasheet" "https://www.mouser.com/datasheet/2/916/BZT52H_Q_SER-2721682.pdf" (id 3) (at 138.43 167.64 0)
       (effects (font (size 1.27 1.27)) hide)
     )
@@
     )
     (path "/5ce8fd98-10c0-4e8c-a1e2-45c9c411680e"
-      (reference "D2") (unit 1) (value "D_Schottky") (footprint "")
+      (reference "D2") (unit 1) (value "D_Schottky") (footprint "Diode_SMD:D_0805_2012Metric")
     )
     (path "/b59f9ec5-7c8d-45b9-9d04-3cc39a39b975"
-      (reference "D3") (unit 1) (value "3.0V±0.05") (footprint "")
+      (reference "D3") (unit 1) (value "3.0V±0.05") (footprint "Diode_SMD:D_0805_2012Metric")
     )
     (path "/aa189804-987d-4086-ae4c-25359c5de72a"

Commit message: shunt connector change
Parts:
- J1: footprint Connector_Molex:Molex_Micro-Fit_3.0_43650-0415_1x04_P3.00mm_Vertical -> Connector_PinSocket_2.54mm:PinSocket_1x05_P2.54mm_Horizontal
Changed lines of the file:
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@@
     (property "Reference" "J1" (id 0) (at 21.1328 116.4082 0))
     (property "Value" "ShuntConn" (id 1) (at 21.1328 118.7196 0))
-    (property "Footprint" "Connector_Molex:Molex_Micro-Fit_3.0_43650-0415_1x04_P3.00mm_Vertical" (id 2) (at 19.05 124.46 0)
+    (property "Footprint" "Connector_PinSocket_2.54mm:PinSocket_1x05_P2.54mm_Horizontal" (id 2) (at 19.05 124.46 0)
       (effects (font (size 1.27 1.27)) hide)
     )
@@
     )
     (path "/00000000-0000-0000-0000-00005f1c3fb3"
-      (reference "J1") (unit 1) (value "ShuntConn") (footprint "Connector_Molex:Molex_Micro-Fit_3.0_43650-0415_1x04_P3.00mm_Vertical")
+      (reference "J1") (unit 1) (value "ShuntConn") (footprint "Connector_PinSocket_2.54mm:PinSocket_1x05_P2.54mm_Horizontal")
     )
     (path "/00000000-0000-0000-0000-00005f0d0a13"

Commit message: mouser 🐁 bom 💣 cart 🛒
Parts:
- C1: Mfg (none) -> TMK212BBJ106MGHT
- C11, C12, C14, C2: Mfg (none) -> UMK212ABJ225KG-T
- C15, C4: Mfg (none) -> C0805C105K5PACTU
- C16: Mfg (none) -> C0805C470JAGACAUTO
- C3: Mfg (none) -> C0805C102J5HACAUTO
- C5: Mfg (none) -> C0805J222K5RACAUTO
- C7: Mfg (none) -> C0805C474K3RAC
- C8, C9: Mfg (none) -> C0805C104M5RACTU
- D1: Mfg (none) -> APTD2012LCGCK
- D2: Mouser# (none) -> RB061QS-20T18R
- D3: Mfg (none) -> BZT52H-A3V0-QX
- R1, R3, R6: Mfg (none) -> CRCW08051K20FKEA
- R2: Mfg (none) -> CRCW08051K50JNEB
- R4: Mfg (none) -> CRCW0805120RFKEA
- R5: Mfg (none) -> CRCW0805806RFKEA
- R7, R8: Mfg (none) -> CRCW080510K0FKEAC
- R9: Mfg (none) -> CRCW080550R0FKTA
- U2: Mfg (none) -> RM-123.3S/H
- U3: Mfg (none) -> LTC6820HMS#PBF
- U4: Mfg (none) -> HX1188FNL
- U6: Mfg (none) -> 584-C2315ITS8-12TMPF
- U7: Mfg (none) -> OPA2196ID
Changed lines of the file:
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@@
+      (effects (font (size 1.27 1.27)) hide)
+    )
+    (property "Mfg" "LTC6820HMS#PBF" (id 4) (at 215.9 46.99 0)
       (effects (font (size 1.27 1.27)) hide)
     )
@@
       (effects (font (size 1.27 1.27)) hide)
     )
+    (property "Mfg" "C0805C104M5RACTU" (id 4) (at 187.96 67.31 0)
+      (effects (font (size 1.27 1.27)) hide)
+    )
     (pin "1")
     (pin "2")
@@
     )
     (property "Datasheet" "https://www.mouser.com/ProductDetail/KEMET/C0805C104M5RACTU?qs=VOOUd%252Bza08qHu13WgNByHQ%3D%3D" (id 3) (at 243.84 72.39 0)
+      (effects (font (size 1.27 1.27)) hide)
+    )
+    (property "Mfg" "C0805C104M5RACTU" (id 4) (at 243.84 72.39 0)
       (effects (font (size 1.27 1.27)) hide)
     )
@@
       (effects (font (size 1.27 1.27)) hide)
     )
+    (property "Mfg" "CRCW08051K20FKEA" (id 4) (at 251.46 52.07 90)
+      (effects (font (size 1.27 1.27)) hide)
+    )
     (pin "1")
     (pin "2")
@@
       (effects (font (size 1.27 1.27)) hide)
     )
+    (property "Mfg" "CRCW0805806RFKEA" (id 4) (at 237.49 49.53 90)
+      (effects (font (size 1.27 1.27)) hide)
+    )
     (pin "1")
     (pin "2")
@@
     )
     (property "Datasheet" "" (id 3) (at 217.17 96.52 0)
+      (effects (font (size 1.27 1.27)) hide)
+    )
+    (property "Mfg" "HX1188FNL" (id 4) (at 217.17 96.52 0)
       (effects (font (size 1.27 1.27)) hide)
     )
@@
       (effects (font (size 1.27 1.27)) hide)
     )
+    (property "Mfg" "CRCW0805120RFKEA" (id 4) (at 185.42 101.6 0)
+      (effects (font (size 1.27 1.27)) hide)
+    )
     (pin "1")
     (pin "2")
@@
       (effects (font (size 1.27 1.27)) hide)
     )
+    (property "Mfg" "TMK212BBJ106MGHT" (id 4) (at 49.53 55.88 0)
+      (effects (font (size 1.27 1.27)) hide)
+    )
     (pin "1")
     (pin "2")
@@
       (effects (font (size 1.27 1.27)) hide)
     )
+    (property "Mfg" "CRCW08051K50JNEB" (id 4) (at 121.92 45.72 0)
+      (effects (font (size 1.27 1.27)) hide)
+    )
     (pin "1")
     (pin "2")
@@
     )
     (property "Datasheet" "~" (id 3) (at 121.92 57.15 0)
+      (effects (font (size 1.27 1.27)) hide)
+    )
+    (property "Mfg" "APTD2012LCGCK" (id 4) (at 121.92 57.15 90)
       (effects (font (size 1.27 1.27)) hide)
     )
@@
       (effects (font (size 1.27 1.27)) hide)
     )
+    (property "Mfg" "C0805C102J5HACAUTO" (id 4) (at 62.23 55.88 0)
+      (effects (font (size 1.27 1.27)) hide)
+    )
     (pin "1")
     (pin "2")
@@
       (effects (font (size 1.27 1.27)) hide)
     )
+    (property "Mfg" "C0805J222K5RACAUTO" (id 4) (at 85.09 67.31 90)
+      (effects (font (size 1.27 1.27)) hide)
+    )
     (pin "1")
     (pin "2")
@@
     )
     (property "Datasheet" "https://www.mouser.com/datasheet/2/468/RO-1711124.pdf" (id 3) (at 85.09 63.5 0)
+      (effects (font (size 1.27 1.27)) hide)
+    )
+    (property "Mfg" "RM-123.3S/H" (id 4) (at 85.09 55.88 0)
       (effects (font (size 1.27 1.27)) hide)
     )
@@
       (effects (font (size 1.27 1.27)) hide)
     )
+    (property "Mfg" "C0805C105K5PACTU" (id 4) (at 21.59 154.94 90)
+      (effects (font (size 1.27 1.27)) hide)
+    )
     (pin "1")
     (pin "2")
@@
       (effects (font (size 1.27 1.27)) hide)
     )
+    (property "Mfg" "CRCW08051K20FKEA" (id 4) (at 50.8 124.46 90)
+      (effects (font (size 1.27 1.27)) hide)
+    )
     (pin "1")
     (pin "2")
@@
       (effects (font (size 1.27 1.27)) hide)
     )
+    (property "Mfg" "CRCW08051K20FKEA" (id 4) (at 50.8 121.92 90)
+      (effects (font (size 1.27 1.27)) hide)
+    )
     (pin "1")
     (pin "2")
@@
     )
     (property "Datasheet" "~" (id 3) (at 58.42 123.19 0)
+      (effects (font (size 1.27 1.27)) hide)
+    )
+    (property "Mfg" "UMK212ABJ225KG-T" (id 4) (at 58.42 123.19 0)
       (effects (font (size 1.27 1.27)) hide)
     )
@@
     )
     (property "Datasheet" "" (id 3) (at 147.32 156.21 0)
+      (effects (font (size 1.27 1.27)) hide)
+    )
+    (property "Mfg" "584-C2315ITS8-12TMPF" (id 4) (at 147.32 156.21 0)
       (effects (font (size 1.27 1.27)) hide)
     )
@@
       (effects (font (size 1.27 1.27)) hide)
     )
+    (property "Mfg" "UMK212ABJ225KG-T" (id 4) (at 167.005 152.4 90)
+      (effects (font (size 1.27 1.27)) hide)
+    )
     (pin "1")
     (pin "2")
@@
       (effects (font (size 1.27 1.27)) hide)
     )
+    (property "Mfg" "UMK212ABJ225KG-T" (id 4) (at 134.62 152.4 90)
+      (effects (font (size 1.27 1.27)) hide)
+    )
     (pin "1")
     (pin "2")
@@
       (effects (font (size 1.27 1.27)) hide)
     )
+    (property "Mfg" "UMK212ABJ225KG-T" (id 4) (at 127 152.4 90)
+      (effects (font (size 1.27 1.27)) hide)
+    )
     (pin "1")
     (pin "2")
@@
     )
     (property "Datasheet" "http://www.ti.com/lit/ds/symlink/opa4196.pdf" (id 3) (at 90.17 151.13 0)
+      (effects (font (size 1.27 1.27)) hide)
+    )
+    (property "Mfg" "OPA2196ID" (id 4) (at 93.98 157.48 0)
       (effects (font (size 1.27 1.27)) hide)
     )
@@
       (effects (font (size 1.27 1.27)) hide)
     )
+    (property "Mfg" "OPA2196ID" (id 4) (at 93.98 157.48 0)
+      (effects (font (size 1.27 1.27)) hide)
+    )
     (pin "1")
     (pin "2")
@@
       (effects (font (size 1.27 1.27)) hide)
     )
+    (property "Mfg" "OPA2196ID" (id 4) (at 93.98 157.48 0)
+      (effects (font (size 1.27 1.27)) hide)
+    )
     (pin "1")
     (pin "2")
@@
       (effects (font (size 1.27 1.27)) hide)
     )
+    (property "Mfg" "C0805C474K3RAC" (id 4) (at 79.375 163.83 0)
+      (effects (font (size 1.27 1.27)) hide)
+    )
     (pin "1")
     (pin "2")
@@
       (effects (font (size 1.27 1.27)) hide)
     )
+    (property "Mfg" "CRCW080510K0FKEAC" (id 4) (at 73.66 157.48 90)
+      (effects (font (size 1.27 1.27)) hide)
+    )
     (pin "1")
     (pin "2")
@@
     )
     (property "Datasheet" "https://www.mouser.com/ProductDetail/KEMET/C0805C105K5PACTU?qs=mYAa4mSiDJyTAfAbrHf%2FRg%3D%3D" (id 3) (at 68.58 151.13 0)
+      (effects (font (size 1.27 1.27)) hide)
+    )
+    (property "Mfg" "C0805C105K5PACTU" (id 4) (at 68.58 151.13 0)
       (effects (font (size 1.27 1.27)) hide)
     )
@@
       (effects (font (size 1.27 1.27)) hide)
     )
+    (property "Mfg" "CRCW080510K0FKEAC" (id 4) (at 62.23 157.48 90)
+      (effects (font (size 1.27 1.27)) hide)
+    )
     (pin "1")
     (pin "2")
@@
     )
     (property "Datasheet" "~" (id 3) (at 130.81 167.64 0)
+      (effects (font (size 1.27 1.27)) hide)
+    )
+    (property "Mfg" "C0805C470JAGACAUTO" (id 4) (at 130.81 167.64 0)
       (effects (font (size 1.27 1.27)) hide)
     )
@@
       (effects (font (size 1.27 1.27)) hide)
     )
+    (property "Mfg" "CRCW080550R0FKTA" (id 4) (at 125.73 160.02 90)
+      (effects (font (size 1.27 1.27)) hide)
+    )
     (pin "1")
     (pin "2")
@@
     )
     (property "Datasheet" "https://fscdn.rohm.com/en/products/databook/datasheet/discrete/diode/schottky_barrier/rb061qs-20-e.pdf" (id 3) (at 44.45 50.8 0)
+      (effects (font (size 1.27 1.27)) hide)
+    )
+    (property "Mouser#" "RB061QS-20T18R" (id 4) (at 44.45 50.8 0)
       (effects (font (size 1.27 1.27)) hide)
     )
@@
       (effects (font (size 1.27 1.27)) hide)
     )
+    (property "Mfg" "BZT52H-A3V0-QX" (id 4) (at 138.43 167.64 90)
+      (effects (font (size 1.27 1.27)) hide)
+    )
