File: BPS-Amperes.kicad_pcb (KiCad board)
At the start: 2 copper layers, 40 x 35 mm, 52 parts, among them J1 ShuntConn, J2 LeaderConn, J3 Conn_01x04, J4 Conn_01x05, U1 INA186A3IDDFT, U2 RO-123.3S_HP, U3 LTC6820, U4 HX1188FNL, U5 REF1930AIDDCT, U6 LTC2315, U7 OPA2196

Commit message: we 👥 do 😳 a little ⌚ graphic designing
Parts:
- moved TP2 2.25 mm to (149.8, 121.0)
Routing:
- net +12V: track 40.6 -> 36.9 mm
Other:
- board text added: "+3V3"
- board text added: "<<< GND PWR"
Changed lines of the file:
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@@
   )
   (footprint "TestPoint:TestPoint_Pad_2.0x2.0mm" (layer "F.Cu")
-    (at 149.75 123.25)
+    (at 149.75 121)
     (descr "SMD rectangular pad as test Point, square 2.0mm side length")
     (tags "test point SMD pad rectangle square")
@@
     )
   )
+  (gr_line (start 118.75 116) (end 121.75 113) (layer "F.SilkS") (width 0.12))
+  (gr_line (start 118.75 113.5) (end 121.75 110.5) (layer "F.SilkS") (width 0.12))
+  (gr_line (start 118.5 122.5) (end 118.5 118.5) (layer "F.SilkS") (width 0.12))
+  (gr_line (start 118.75 108.5) (end 121.5 105.75) (layer "F.SilkS") (width 0.12))
+  (gr_line (start 118.75 111) (end 122 107.75) (layer "F.SilkS") (width 0.12))
   (gr_line (start 155 99) (end 155 126) (layer "Edge.Cuts") (width 0.05))
   (gr_arc (start 155 126) (mid 153.828427 128.828427) (end 151 130) (layer "Edge.Cuts") (width 0.05))
@@
     (effects (font (size 1 1) (thickness 0.15)) (justify mirror))
   )
-  (gr_text "test" (at 149.8 112.6) (layer "F.SilkS")
+  (gr_text "test" (at 149.75 112.6) (layer "F.SilkS")
     (effects (font (size 1 1) (thickness 0.2)))
   )
@@
     (effects (font (size 1 1) (thickness 0.2)))
   )
-  (gr_text "+12V" (at 146.5 126) (layer "F.SilkS")
-    (effects (font (size 1 1) (thickness 0.15)))
-  )
-  (gr_text "IP" (at 133 123) (layer "F.SilkS")
+  (gr_text "+12V" (at 152 126 90) (layer "F.SilkS")
     (effects (font (size 0.8 0.8) (thickness 0.15)))
   )
-  (gr_text "shunt\n" (at 149.4 110.4) (layer "F.SilkS")
+  (gr_text "IP" (at 133.25 123) (layer "F.SilkS")
+    (effects (font (size 1 1) (thickness 0.2)))
+  )
+  (gr_text "shunt\n" (at 149 110.4) (layer "F.SilkS")
     (effects (font (size 1 1) (thickness 0.2)))
   )
-  (gr_text "R-" (at 150.2 117.4) (layer "F.SilkS")
+  (gr_text "R-" (at 150 117.4) (layer "F.SilkS")
     (effects (font (size 1 1) (thickness 0.2)))
   )
-  (gr_text "ETS" (at 120.5 107.5 45) (layer "F.SilkS")
+  (gr_text "ETS" (at 120.25 106 45) (layer "F.SilkS")
     (effects (font (size 0.8 0.8) (thickness 0.15)))
   )
@@
     (effects (font (size 0.8 0.8) (thickness 0.15)))
   )
+  (gr_text "GND" (at 120.25 113.5 45) (layer "F.SilkS")
+    (effects (font (size 0.8 0.8) (thickness 0.15)))
+  )
   (gr_text "GND" (at 131.2 100.8 90) (layer "F.SilkS")
     (effects (font (size 1 1) (thickness 0.2)))
   )
   (gr_text "IM" (at 135.5 123) (layer "F.SilkS")
-    (effects (font (size 0.8 0.8) (thickness 0.15)))
+    (effects (font (size 1 1) (thickness 0.2)))
   )
-  (gr_text "RSHL" (at 120.5 112.5 45) (layer "F.SilkS")
+  (gr_text "RSHL" (at 120.5 110.75 45) (layer "F.SilkS")
     (effects (font (size 0.8 0.8) (thickness 0.15)))
   )
-  (gr_text "GND\nPWR" (at 152.5 123.25) (layer "F.SilkS")
+  (gr_text "GND\nPWR" (at 152.5 121) (layer "F.SilkS")
     (effects (font (size 0.8 0.8) (thickness 0.15)))
   )
@@
     (effects (font (size 0.8 0.8) (thickness 0.15)))
   )
-  (gr_text "RSHH" (at 120.5 110 45) (layer "F.SilkS")
+  (gr_text "<<<\nGND\nPWR" (at 145.25 126.25) (layer "F.SilkS")
+    (effects (font (size 1 1) (thickness 0.2)))
+  )
+  (gr_text "RSHH" (at 120.5 108.25 45) (layer "F.SilkS")
     (effects (font (size 0.8 0.8) (thickness 0.15)))
   )
@@
     (effects (font (size 1 1) (thickness 0.2)))
   )
-  (gr_text "R+" (at 150.2 115) (layer "F.SilkS")
+  (gr_text "R+" (at 150 115) (layer "F.SilkS")
+    (effects (font (size 1 1) (thickness 0.2)))
+  )
+  (gr_text "+12V" (at 130.5 121.75 90) (layer "F.SilkS")
     (effects (font (size 1 1) (thickness 0.2)))
   )
-  (gr_text "+12V" (at 129.5 123) (layer "F.SilkS")
+  (gr_text "+3V3" (at 117.75 121 90) (layer "F.SilkS")
     (effects (font (size 0.8 0.8) (thickness 0.15)))
   )
@@
   (segment (start 144.05 103.86) (end 143.69 103.5) (width 0.4) (layer "F.Cu") (net 1))
   (segment (start 144 106.85) (end 144.05 106.8) (width 0.4) (layer "F.Cu") (net 1))
+  (segment (start 149.75 121) (end 149.75 121.75) (width 0.2) (layer "F.Cu") (net 1))
   (segment (start 144.05 106.8) (end 144.05 103.86) (width 0.4) (layer "F.Cu") (net 1))
-  (segment (start 149 120.75) (end 149 122.5) (width 0.2) (layer "F.Cu") (net 1))
-  (segment (start 149 122.5) (end 149.75 123.25) (width 0.2) (layer "F.Cu") (net 1))
+  (segment (start 149.75 121.75) (end 148.625 122.875) (width 0.2) (layer "F.Cu") (net 1))
   (segment (start 144 108.8) (end 144 106.85) (width 0.4) (layer "F.Cu") (net 1))
-  (via (at 149 120.75) (size 0.8) (drill 0.4) (layers "F.Cu" "B.Cu") (net 1))
+  (via (at 148.625 122.875) (size 0.8) (drill 0.4) (layers "F.Cu" "B.Cu") (net 1))
   (segment (start 142.079 101.889) (end 142.079 99) (width 1) (layer "B.Cu") (net 1))
   (segment (start 141.415 124) (end 147.5 124) (width 1) (layer "B.Cu") (net 1))
+  (segment (start 148.625 122.875) (end 149 122.5) (width 1) (layer "B.Cu") (net 1))
   (segment (start 149 113.5) (end 143.69 108.19) (width 1) (layer "B.Cu") (net 1))
-  (segment (start 147.5 124) (end 149 122.5) (width 1) (layer "B.Cu") (net 1))
+  (segment (start 147.5 124) (end 148.625 122.875) (width 1) (layer "B.Cu") (net 1))
   (segment (start 149 120.75) (end 149 113.5) (width 1) (layer "B.Cu") (net 1))
   (segment (start 149 122.5) (end 149 120.75) (width 1) (layer "B.Cu") (net 1))
@@
   (segment (start 139.5 125.915) (end 141.415 124) (width 1) (layer "B.Cu") (net 1))
   (segment (start 143.69 103.5) (end 142.079 101.889) (width 1) (layer "B.Cu") (net 1))
-  (segment (start 150.977 124.523) (end 149.75 125.75) (width 0.2) (layer "F.Cu") (net 2))
-  (segment (start 150.25 120.75) (end 150.977 121.477) (width 0.2) (layer "F.Cu") (net 2))
-  (segment (start 150.977 121.477) (end 150.977 124.523) (width 0.2) (layer "F.Cu") (net 2))
+  (segment (start 149.75 124) (end 149.5 123.75) (width 0.2) (layer "F.Cu") (net 2))
   (segment (start 145.95 106.8) (end 145.95 103.78) (width 0.4) (layer "F.Cu") (net 2))
   (segment (start 145.95 103.78) (end 146.23 103.5) (width 0.4) (layer "F.Cu") (net 2))
-  (via (at 150.25 120.75) (size 0.8) (drill 0.4) (layers "F.Cu" "B.Cu") (net 2))
+  (segment (start 149.75 125.75) (end 149.75 124) (width 0.2) (layer "F.Cu") (net 2))
+  (via (at 149.5 123.75) (size 0.8) (drill 0.4) (layers "F.Cu" "B.Cu") (net 2))
   (segment (start 150.25 113) (end 146.23 108.98) (width 1) (layer "B.Cu") (net 2))
   (segment (start 146.23 103.5) (end 147.921 101.809) (width 1) (layer "B.Cu") (net 2))
   (segment (start 146.23 108.98) (end 146.23 103.5) (width 1) (layer "B.Cu") (net 2))
-  (segment (start 147.25 126) (end 150.25 123) (width 1) (layer "B.Cu") (net 2))
+  (segment (start 147.25 126) (end 149.5 123.75) (width 1) (layer "B.Cu") (net 2))
+  (segment (start 149.5 123.75) (end 150.25 123) (width 1) (layer "B.Cu") (net 2))
   (segment (start 147.921 101.809) (end 147.921 99) (width 1) (layer "B.Cu") (net 2))
   (segment (start 150.25 120.75) (end 150.25 113) (width 1) (layer "B.Cu") (net 2))
@@
     (polygon
       (pts
-        (xy 141.25 112.25)
-        (xy 134.25 112.25)
+        (xy 141.25 105.5)
+        (xy 136.25 105.5)
+        (xy 136.25 108)
+        (xy 136.25 108.75)
+        (xy 136.25 113.75)
+        (xy 134.25 113.75)
         (xy 134.25 123.5)
         (xy 126.5 123.5)

Commit message: womp womp
Parts:
- removed C1: 10u, UTSVT_Passive:C_2220_5750Metrix
- removed C10, C15, C18, C4: 1uF, Capacitor_SMD:C_0805_2012Metric
- removed C11, C12, C14, C2: 2.2uF, Capacitor_SMD:C_0805_2012Metric
- removed C13, C17, C6: 100nF, Capacitor_SMD:C_0805_2012Metric
- removed C16: 47pF, Capacitor_SMD:C_0805_2012Metric
- removed C3: 1n, Capacitor_SMD:C_0805_2012Metric
- removed C5: 2.2n, Capacitor_SMD:C_0805_2012Metric
- removed C7: 470nF, Capacitor_SMD:C_0805_2012Metric
- removed C8, C9: 0.1u, Capacitor_SMD:C_0805_2012Metric
- removed D1: PowerOn, LED_SMD:LED_0805_2012Metric
- removed D2: D_Schottky, Diode_SMD:D_0805_2012Metric
- removed D3: 3.0V±0.05, Diode_SMD:D_0805_2012Metric
- removed FB1, FB2: FerriteBead_Small, Inductor_SMD:L_0805_2012Metric
- removed J1: ShuntConn, Connector_PinSocket_2.54mm:PinSocket_1x05_P2.54mm_Vertical
- removed J2: LeaderConn, Connector_Molex:Molex_Micro-Fit_3.0_43650-0415_1x04_P3.00mm_Vertical
- removed J3: Conn_01x04, Connector_PinHeader_2.54mm:PinHeader_1x04_P2.54mm_Vertical
- removed J4: Conn_01x05, Connector_PinHeader_2.54mm:PinHeader_1x05_P2.54mm_Vertical
- removed R1, R3: 1.2k, Resistor_SMD:R_0805_2012Metric
- removed R2: 1.5k, Resistor_SMD:R_0805_2012Metric
- removed R4: 120, Resistor_SMD:R_0805_2012Metric
- removed R5: 806, Resistor_SMD:R_0805_2012Metric
- removed R6: 1.21k, Resistor_SMD:R_0805_2012Metric
- removed R7, R8: 10k, Resistor_SMD:R_0805_2012Metric
- removed R9: 50, Resistor_SMD:R_0805_2012Metric
- removed TP1: +12V_TP, TestPoint:TestPoint_Pad_2.0x2.0mm
- removed TP2: GNDPWR_TP, TestPoint:TestPoint_Pad_2.0x2.0mm
- removed TP3: +3.3V_TP, TestPoint:TestPoint_Pad_1.5x1.5mm
- removed TP4: GND_TP, TestPoint:TestPoint_Pad_1.5x1.5mm
- removed TP5: Ain_TP, Connector_PinSocket_2.54mm:PinSocket_1x01_P2.54mm_Vertical
- removed TP6: +1V5_TP, TestPoint:TestPoint_Pad_1.5x1.5mm
- removed TP7: +3V0_TP, TestPoint:TestPoint_Pad_1.5x1.5mm
- removed U1: INA186A3IDDFT, Package_TO_SOT_SMD:SOT-23-8
- removed U2: RO-123.3S_HP, UTSVT_ICs:RI3_DC_Converter
- removed U3: LTC6820, Package_SO:MSOP-16_3x4mm_P0.5mm
- removed U4: HX1188FNL, UTSVT_Passive:HXXXX
- removed U5: REF1930AIDDCT, Package_TO_SOT_SMD:SOT-23-5
- removed U6: LTC2315, Package_TO_SOT_SMD:SOT-23-8
- removed U7: OPA2196, Package_SO:SOIC-8_3.9x4.9mm_P1.27mm
Routing:
- net +3V3: track 108.8 -> 0.00 mm, vias 4 -> 0
- net GND: track 49.9 -> 0.00 mm, vias 41 -> 0
- net +3V0: track 48.7 -> 0.00 mm, vias 4 -> 0
- net GNDPWR: track 45.1 -> 0.00 mm, vias 1 -> 0
- net +12V: track 36.9 -> 0.00 mm, vias 1 -> 0
- net +1V5: track 34.8 -> 0.00 mm, vias 1 -> 0
- net /MISO: track 20.7 -> 0.00 mm, vias 1 -> 0
- net /SCK: track 18.5 -> 0.00 mm, vias 1 -> 0
- net /CS: track 18.0 -> 0.00 mm, vias 1 -> 0
- net /+12V_In: track 15.8 -> 0.00 mm
- net Net-(J2-Pad3): track 15.5 -> 0.00 mm
- net /IP: track 12.6 -> 0.00 mm
- net Net-(C16-Pad1): track 10.2 -> 0.00 mm
- net Net-(C15-Pad2): track 10.1 -> 0.00 mm
- net Net-(J2-Pad2): track 8.86 -> 0.00 mm
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- removed copper zone on B.Cu, net GND
- removed copper zone on F.Cu, net GND
Other:
- board outline removed
- board text removed: "+12V"
- board text removed: "+3V3"
- board text removed: "1v5"
- board text removed: "3v0"
- board text removed: "3v3"
- board text removed: "<<< GND PWR"
- board text removed: "CS"
- board text removed: "ETS"
- board text removed: "GND"
- board text removed: "GND PWR"
- board text removed: "IM"
- board text removed: "IP"
- board text removed: "MISO"
- board text removed: "Manthan approved this pull request. github.com/ manthanand"
- board text removed: "R+"
- board text removed: "R-"
- board text removed: "RSHH"
- board text removed: "RSHL"
- board text removed: "SCK"
- board text removed: "shunt"
- board text removed: "test"
